Commit message: enabled visualization with rviz2

File: robotic_arm/urdf/robotic_arm.urdf (robot description, URDF)
Before this commit: robot robotic_arm, 7 links, 6 joints
Links:
- removed link Link_1
- removed link Link_2
- removed link Link_3
- removed link Link_4
- removed link Link_5
- removed link Link_6
- added link end_effector, mass 0.0505964546832365; collision mesh filename=package://robotic_arm/meshes/end_effector.STL; visual mesh filename=package://robotic_arm/meshes/end_effector.STL
- added link link_1, mass 0.0465317343320066; collision mesh filename=package://robotic_arm/meshes/link_1.STL; visual mesh filename=package://robotic_arm/meshes/link_1.STL
- added link link_2, mass 0.0196331437668373; collision mesh filename=package://robotic_arm/meshes/link_2.STL; visual mesh filename=package://robotic_arm/meshes/link_2.STL
- added link link_3, mass 0.0527193093583245; collision mesh filename=package://robotic_arm/meshes/link_3.STL; visual mesh filename=package://robotic_arm/meshes/link_3.STL
- added link link_4, mass 0.0734303248905977; collision mesh filename=package://robotic_arm/meshes/link_4.STL; visual mesh filename=package://robotic_arm/meshes/link_4.STL
- link base_link: mass None -> 0.0953444546366154; geometry collision mesh filename=package://robotic_arm/meshes/base_link.STL; visual mesh filename=package://robotic_arm/meshes/base_link.STL
Joints:
- removed joint Joint_1
- removed joint Joint_2
- removed joint Joint_3
- removed joint Joint_4
- removed joint Joint_5
- removed joint base_to_link1
- added joint end_effector_joint: type continuous, parent link_4, child end_effector, origin xyz=0.00668895775777986 0.015904071986752 0.0405109050654748 rpy=2.00026591436005 0.0503809083594157 -3.01899503858886, axis 0.0765333432788003 -0.713482347733641 -0.696480858917932
- added joint joint_1: type continuous, parent base_link, child link_1, origin xyz=0.681512899942898 -1.31957371207269 0.9106277233023 rpy=1.57079632679489 0 2.38986902292884, axis 0 1 0
- added joint joint_2: type continuous, parent link_1, child link_2, origin xyz=-0.0138083245935132 0.0680000000000357 -0.0144682470230319 rpy=0.244836805062138 -0.375384253365743 -3.01423665910926, axis 0.920715361532491 0.00279090919548123 0.390224850392638
- added joint joint_3: type continuous, parent link_2, child link_3, origin xyz=-0.0119074417180245 -0.0981728744550843 0.0287975674968496 rpy=0.666909771133124 0.72745528612343 -2.87911848216658, axis 0.920648187108123 0.00215985289631251 0.39038730846429
- added joint joint_4: type continuous, parent link_3, child link_4, origin xyz=0.00878557193452059 0.0942863948809806 -0.0213160274783319 rpy=2.98177224561093 0.0793264831605607 -3.13671933164858, axis 0.951231015101866 -0.0451134015264731 0.305162803944034
